Commit message: rviz display

File: urdf/fred_montagem.urdf (robot description, URDF)
Before this commit: robot fred_montagem, 5 links, 4 joints
Links:
- removed link wheel1
- removed link wheel2
- removed link wheel3
- removed link wheel4
- added link base_footprint; visual box size=0.001 0.001 0.001
- added link lidar_link
- added link roda1_link, mass 0.429989283650456; collision mesh filename=package://fred_montagem/meshes/roda1.STL; visual mesh filename=package://fred_montagem/meshes/roda1.STL
- added link roda2, mass 0.429989283650456; collision mesh filename=package://fred_montagem/meshes/roda2.STL; visual mesh filename=package://fred_montagem/meshes/roda2.STL
- added link roda3, mass 0.429989283650456; collision mesh filename=package://fred_montagem/meshes/roda3.STL; visual mesh filename=package://fred_montagem/meshes/roda3.STL
- added link roda4, mass 0.429989283650456; collision mesh filename=package://fred_montagem/meshes/roda4.STL; visual mesh filename=package://fred_montagem/meshes/roda4.STL
- link base_link: mass 4.6314332951117 -> 4.63143329848068
Joints:
- removed joint joint1
- removed joint joint2
- removed joint joint3
- removed joint joint4
- added joint base_link_to_base_footprint: type fixed, parent base_footprint, child base_link, origin xyz=0 0 0.1 rpy=0 0 0
- added joint lidar_joint: type fixed, parent base_link, child lidar_link, origin xyz=0 0.18 0.187 rpy=0 0 0
- added joint roda1: type continuous, parent base_link, child roda1_link, origin xyz=0.14881 0.113 0.025 rpy=1.5708 -1.3493 1.5708, axis 0 0 1
- added joint roda2: type continuous, parent base_link, child roda2, origin xyz=-0.14881 0.113 0.025 rpy=1.5708 1.3493 -1.5708, axis 0 0 1
- added joint roda3: type continuous, parent base_link, child roda3, origin xyz=0.14881 -0.113 0.025 rpy=1.5708 0.72582 1.5708, axis 0 0 1
- added joint roda4: type continuous, parent base_link, child roda4, origin xyz=-0.14881 -0.113 0.025 rpy=1.5708 -0.72582 -1.5708, axis 0 0 1

Commit message: retirando base_footptint

File: urdf/fred_montagem.urdf (robot description, URDF)
Before this commit: robot fred_montagem, 7 links, 6 joints
Links:
- removed link base_footprint
Joints:
- removed joint base_link_to_base_footprint
